Commit message: collision details

File: description/robot_core.xacro (robot description, xacro)
@@ -28,4 +28,69 @@
         <material name="white"/>
     </visual>
+    <collision>
+        <origin xyz="0.15 0 0.075" rpy="0 0 0"/>
+        <geometry>
+            <box size="0.3 0.3 0.15"/>
+        </geometry>
+    </collision>
+</link>
+<joint name="left_wheel_joint" type="continuous">
+    <parent link="base_link"/>
+    <child link="left_wheel"/>
+    <origin xyz="0 0.175 0" rpy="-${pi/2} 0 0"/>
+    <axis xyz="0 0 1"/>
+</joint>
+<link name="left_wheel">
+    <visual>
+        <geometry>
+            <cylinder length="0.04" radius="0.05" />
+        </geometry>
+        <material name="blue"/>
+    </visual>
+    <collision>
+        <geometry>
+            <cylinder length="0.04" radius="0.05" />
+        </geometry>
+        <material name="blue"/>
+    </collision>
+</link>
+<joint name="right_wheel_joint" type="continuous">
+    <parent link="base_link"/>
+    <child link="right_wheel"/>
+    <origin xyz="0 -0.175 0" rpy="${pi/2} 0 0"/>
+    <axis xyz="0 0 -1"/>
+</joint>
+<link name="right_wheel">
+    <visual>
+        <geometry>
+            <cylinder length="0.04" radius="0.05" />
+        </geometry>
+        <material name="blue"/>
+    </visual>
+    <collision>
+        <geometry>
+            <cylinder length="0.04" radius="0.05" />
+        </geometry>
+        <material name="blue"/>
+    </collision>
+</link>
+<joint name="caster_wheel_joint" type="fixed">
+    <parent link="chassis"/>
+    <child link="caster_wheel"/>
+    <origin xyz="0.24 0 0" rpy="0 0 0"/>
+</joint>
+<link name="caster_wheel">
+    <visual>
+        <geometry>
+            <sphere radius="0.05" />
+        </geometry>
+        <material name="black"/>
+    </visual>
+    <collision>
+        <geometry>
+            <sphere radius="0.05" />
+        </geometry>
+        <material name="black"/>
+    </collision>
 </link>
 </robot>

Commit message: inertia

File: description/robot_core.xacro (robot description, xacro)
@@ -94,3 +94,27 @@
     </collision>
 </link>
+<link name="chassis">
+     <!-- ... visual and collision here ... -->
+    <xacro:inertial_box mass="0.5" x="0.3" y="0.3" z="0.15">
+        <origin xyz="0.15 0 0.075" rpy="0 0 0"/>
+    </xacro:inertial_box>
+</link>
+<link name="left_wheel">
+    <!-- ... visual and collision here ... -->
+    <xacro:inertial_cylinder mass="0.1" length="0.05" radius="0.05">
+        <origin xyz="0 0 0" rpy="0 0 0"/>
+    </xacro:inertial_cylinder>
+</link>
+<link name="right_wheel">
+    <!-- ... visual and collision here ... -->
+    <xacro:inertial_cylinder mass="0.1" length="0.05" radius="0.05">
+        <origin xyz="0 0 0" rpy="0 0 0"/>
+    </xacro:inertial_cylinder>
+</link>
+<link name="caster_wheel">
+    <!-- ... visual and collision here ... -->
+    <xacro:inertial_sphere mass="0.1" radius="0.05">
+        <origin xyz="0 0 0" rpy="0 0 0"/>
+    </xacro:inertial_sphere>
+</link>
 </robot>

Commit message: fixing robot core

File: description/robot_core.xacro (robot description, xacro)
@@ -1,4 +1,5 @@
 <?xml version="1.0"?>
 <robot xmlns:xacro="http://www.ros.org/wiki/xacro">
+<xacro:include filename="inertial_macros.xacro" />
     <material name="white">
     <color rgba="1 1 1 1"/>
@@ -34,4 +35,7 @@
         </geometry>
     </collision>
+        <xacro:inertial_box mass="0.5" x="0.3" y="0.3" z="0.15">
+        <origin xyz="0.15 0 0.075" rpy="0 0 0"/>
+    </xacro:inertial_box>
 </link>
 <joint name="left_wheel_joint" type="continuous">
@@ -54,4 +58,7 @@
         <material name="blue"/>
     </collision>
+    <xacro:inertial_cylinder mass="0.1" length="0.05" radius="0.05">
+        <origin xyz="0 0 0" rpy="0 0 0"/>
+    </xacro:inertial_cylinder>
 </link>
 <joint name="right_wheel_joint" type="continuous">
@@ -74,4 +81,7 @@
         <material name="blue"/>
     </collision>
+    <xacro:inertial_cylinder mass="0.1" length="0.05" radius="0.05">
+        <origin xyz="0 0 0" rpy="0 0 0"/>
+    </xacro:inertial_cylinder>
 </link>
 <joint name="caster_wheel_joint" type="fixed">
@@ -93,25 +103,4 @@
         <material name="black"/>
     </collision>
-</link>
-<link name="chassis">
-     <!-- ... visual and collision here ... -->
-    <xacro:inertial_box mass="0.5" x="0.3" y="0.3" z="0.15">
-        <origin xyz="0.15 0 0.075" rpy="0 0 0"/>
-    </xacro:inertial_box>
-</link>
-<link name="left_wheel">
-    <!-- ... visual and collision here ... -->
-    <xacro:inertial_cylinder mass="0.1" length="0.05" radius="0.05">
-        <origin xyz="0 0 0" rpy="0 0 0"/>
-    </xacro:inertial_cylinder>
-</link>
-<link name="right_wheel">
-    <!-- ... visual and collision here ... -->
-    <xacro:inertial_cylinder mass="0.1" length="0.05" radius="0.05">
-        <origin xyz="0 0 0" rpy="0 0 0"/>
-    </xacro:inertial_cylinder>
-</link>
-<link name="caster_wheel">
-    <!-- ... visual and collision here ... -->
     <xacro:inertial_sphere mass="0.1" radius="0.05">
         <origin xyz="0 0 0" rpy="0 0 0"/>

Commit message: gazebo chassis

File: description/robot_core.xacro (robot description, xacro)
@@ -107,3 +107,6 @@
     </xacro:inertial_sphere>
 </link>
+<gazebo reference="chassis">
+    <material>Gazebo/White</material>
+</gazebo>
 </robot>

Commit message: castor wheel gazebo

File: description/robot_core.xacro (robot description, xacro)
@@ -110,3 +110,8 @@
     <material>Gazebo/White</material>
 </gazebo>
+<gazebo reference="caster_wheel">
+    <material>Gazebo/Black</material>
+    <mu1 value="0.001"/>
+    <mu2 value="0.001"/>
+</gazebo>
 </robot>
